File: pcb/pro/Ntester/InStage.sch (KiCad schematic (older format))
At the start: 13 parts

Commit message: added rest of files
Parts:
- removed C?: 330uF, symbol Device:CP_Small
- removed C?: DNP, symbol Device:CP_Small
- removed R? (x3): 1k, symbol Device:R_Small
- removed R?: 470R, symbol Device:R_Small
- added C1, C12, C13, C3: B45196-H2227-M409, Capacitor_Tantalum_SMD:CP_EIA-7343-31_Kemet-D, symbol Device:CP_Small
- added C10, C11, C15, C16: 0603B104M500CT, Resistor_SMD:R_0603_1608Metric, symbol Device:C_Small
- added C14: DNP, Capacitor_Tantalum_SMD:CP_EIA-7343-31_Kemet-D, symbol Device:CP_Small
- added R1: RNCF0603TKY250R, Resistor_SMD:R_0603_1608Metric, symbol Device:R_Small
- added R2: RNCF0603AKT10R0, Resistor_SMD:R_0603_1608Metric, symbol Device:R_Small
- added R5: CR0603-JW-471ELF, Resistor_SMD:R_0603_1608Metric, symbol Device:R_Small
- added RN1: ACASA1001S1001P1AT, Resistor_SMD:R_Array_Convex_4x1206, symbol Device:R_Pack04
- C8: renamed from C?; value 100p -> 885012006038; footprint (none) -> Resistor_SMD:R_0603_1608Metric
- C9: renamed from C?; value 68p -> 885012006007; footprint (none) -> Resistor_SMD:R_0603_1608Metric
- Q1: renamed from Q?; value BC847BDW1 -> BC847BDW1T1G
- R4: renamed from R?; value 470R -> CR0603-JW-471ELF; footprint (none) -> Resistor_SMD:R_0603_1608Metric
- R6: renamed from R?; value R_Small -> RG1608N-101-W-T1; footprint (none) -> Resistor_SMD:R_0603_1608Metric
- U1: renamed from U?; footprint (none) -> Package_SO:MSOP-8_3x3mm_P0.65mm
Connections:
- net +5V: now also U1.7 (V+), C10.1, C16.1, C3.1, RN1.5 (R4.2), RN1.6 (R3.2)
- net -5V: now also U1.4 (V-), C1.2, C11.2, C15.2, RN1.8 (R1.2)
- net IN_SIG: now also Q1.2 (B1), RN1.2 (R2.1), RN1.7 (R2.2)
- net at U1.3 (+): now also R5.1
- net at C9.1, U1.6: now also C12.1, C13.1, C14.1, R1.2
- net R_LTP5: now reaches Q1.1 (E1), Q1.4 (E2)
- net R_LTP5: now also RN1.1 (R1.1)
- net R_LTP0: now reaches C8.2, Q1.6 (C1), R4.2
- net R_LTP0: now also RN1.4 (R4.1)
- net R_LTP2: now reaches C8.1, Q1.3 (C2)
- net R_LTP2: now also R5.2, RN1.3 (R3.1)
- net at Q1.5 (B2): now also R1.1, R2.2
- net at R6.2: now also C12.2, C13.2, C14.2
- new net GND: C1.1, C10.2, C11.1, C15.1, C16.2, C3.2, R2.1
Other:
- note added: "100n"
- note added: "100p"
- note added: "10R"
- note added: "220uF/10V"
- note added: "250R"
- note added: "470R"
- note added: "68p"
- note added: "Checklist:\n-thermals (resistor nietwork will be hot)\n-thermocopule junctions"
- note added: "Long tail pair bypassing\n"
- moved on the sheet: C8, C9, Q1A, Q1B, R4, R6, U1

Commit message: " alomost" finalized layout
Parts:
- removed C1, C12, C13, C3: B45196-H2227-M409, Capacitor_Tantalum_SMD:CP_EIA-7343-31_Kemet-D, symbol Device:CP_Small
- removed C10, C11, C15, C16: 0603B104M500CT, Resistor_SMD:R_0603_1608Metric, symbol Device:C_Small
- removed C14: DNP, Capacitor_Tantalum_SMD:CP_EIA-7343-31_Kemet-D, symbol Device:CP_Small
- removed C8: 885012006038, Resistor_SMD:R_0603_1608Metric, symbol Device:C_Small
- removed C9: 885012006007, Resistor_SMD:R_0603_1608Metric, symbol Device:C_Small
- removed Q1: BC847BDW1T1G, Package_TO_SOT_SMD:SOT-363_SC-70-6, symbol Transistor_BJT:BC847BDW1
- removed R1: RNCF0603TKY250R, Resistor_SMD:R_0603_1608Metric, symbol Device:R_Small
- removed R2: RNCF0603AKT10R0, Resistor_SMD:R_0603_1608Metric, symbol Device:R_Small
- removed R4, R5: CR0603-JW-471ELF, Resistor_SMD:R_0603_1608Metric, symbol Device:R_Small
- removed R6: RG1608N-101-W-T1, Resistor_SMD:R_0603_1608Metric, symbol Device:R_Small
- removed RN1: ACASA1001S1001P1AT, Resistor_SMD:R_Array_Convex_4x1206, symbol Device:R_Pack04
- removed U1: LT1818, Package_SO:MSOP-8_3x3mm_P0.65mm, symbol Ntester_additional:LT1818
- added C2: 885012006007, Resistor_SMD:R_0603_1608Metric, symbol Device:C_Small
- added C22, C6, C7: B45196-H2227-M409, Capacitor_Tantalum_SMD:CP_EIA-7343-31_Kemet-D, symbol Device:CP_Small
- added C23: DNP, Capacitor_Tantalum_SMD:CP_EIA-7343-31_Kemet-D, symbol Device:CP_Small
- added C4, C5: 0603B104M500CT, Resistor_SMD:R_0603_1608Metric, symbol Device:C_Small
- added D1, D2: BAS116LT1G, Package_TO_SOT_SMD:SOT-23, symbol Device:D_Schottky_AAK
- added FB1: 742792651, Resistor_SMD:R_0603_1608Metric, symbol Device:Ferrite_Bead_Small
- added J4: 67996-408HLF, Connector_PinHeader_2.54mm:PinHeader_2x04_P2.54mm_Vertical, symbol Connector_Generic:Conn_02x04_Odd_Even
- added JP1: CAL_FUSE, Jumper:SolderJumper-2_P1.3mm_Bridged_Pad1.0x1.5mm, symbol Device:Jumper_NC_Small
- added R3: RHC2512FT4R99, Resistor_SMD:R_2512_6332Metric, symbol Device:R_Small
- added R7: CRM2512-JW-470ELF, Resistor_SMD:R_2512_6332Metric, symbol Device:R_Small
- added R8: CR1206-FX-4990ELF, Resistor_SMD:R_1206_3216Metric, symbol Device:R_Small
- added R9: RMCF0603FT499R, Resistor_SMD:R_0603_1608Metric, symbol Device:R_Small
Connections:
- net +5V: now also C4.1, D1.3 (K)
- net -5V: now also C5.1, D2.3 (K)
- net GND: now also C2.2, C4.2, C5.2, JP1.2, R3.2, R7.2, R8.2, R9.2
- new net: C2.1, C22.1, C23.1, C6.1, C7.1, D1.1 (A), D2.1 (A), FB1.1, J4.1 (Pin_1), J4.3 (Pin_3), J4.5 (Pin_5), J4.7 (Pin_7)
- new net: J4.6 (Pin_6), R7.1
- new net: J4.8 (Pin_8), R3.1
- new net: J4.4 (Pin_4), R8.1
- new net: J4.2 (Pin_2), JP1.1
- new net IN_STG: FB1.2
- new net OUT_STG: C22.2, C23.2, C6.2, C7.2, R9.1
- no-connect marks 0 -> 2
Other:
- note added: "0R - cal only\n5R -> 2A -> 20W\n50R -> 200mA -> 2W\n499R -> 20mA -> 0.2W"
- note added: "499R"
- note removed: "100n"
- note removed: "100p"
- note removed: "10R"
- note removed: "250R"
- note removed: "470R"
- note removed: "Checklist:\n-thermals (resistor nietwork will be hot)\n-thermocopule junctions"
- note removed: "Long tail pair bypassing\n"

Commit message: layout finalized
Connections:
- net -5V: now also D2.1 (A); no longer D2.3 (K)
- net at C2.1, C22.1, C23.1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: now also D2.3 (K); no longer D2.1 (A)
Other:
- moved on the sheet: C5, D2
Changed lines of the file:
@@
 $Descr A4 11693 8268
 encoding utf-8
-Sheet 4 5
-Title ""
+Sheet 4 8
+Title "Power Supply Noise Tester"
 Date ""
-Rev ""
-Comp ""
+Rev "1.0"
+Comp "Paweł Woźny"
 Comment1 ""
 Comment2 ""
@@
 L Device:D_Schottky_AAK D?
 U 1 1 5BD8662D
-P 4150 3550
+P 4150 3450
 AR Path="/5BD8662D" Ref="D?"  Part="1"
 AR Path="/5BD77D91/5BD8662D" Ref="D2"  Part="1"
-F 0 "D2" V 4129 3694 50  0000 L CNN
-F 1 "BAS116LT1G" V 4220 3694 50  0000 L CNN
-F 2 "Package_TO_SOT_SMD:SOT-23" H 4150 3550 50  0001 C CNN
-F 3 "http://www.onsemi.com/pub/Collateral/BAS116LT1-D.PDF" H 4150 3550 50  0001 C CNN
-	1    4150 3550
-	0    1    -1   0
-$EndComp
-NoConn ~ 4150 3350
-Wire Wire Line
-	4150 3700 4150 3800
+F 0 "D2" V 4129 3594 50  0000 L CNN
+F 1 "BAS116LT1G" V 4220 3594 50  0000 L CNN
+F 2 "Package_TO_SOT_SMD:SOT-23" H 4150 3450 50  0001 C CNN
+F 3 "http://www.onsemi.com/pub/Collateral/BAS116LT1-D.PDF" H 4150 3450 50  0001 C CNN
+	1    4150 3450
+	0    1    1    0
+$EndComp
+Wire Wire Line
+	4250 3650 4250 3800
 $Comp
 L power:-5V #PWR?
 U 1 1 5BD86635
-P 4150 3850
+P 4250 3850
 AR Path="/5BCA1695/5BD86635" Ref="#PWR?"  Part="1"
 AR Path="/5BE0B501/5BD86635" Ref="#PWR?"  Part="1"
 AR Path="/5BD86635" Ref="#PWR?"  Part="1"
 AR Path="/5BD77D91/5BD86635" Ref="#PWR0138"  Part="1"
-F 0 "#PWR0138" H 4150 3950 50  0001 C CNN
-F 1 "-5V" H 4165 4023 50  0000 C CNN
-F 2 "" H 4150 3850 50  0001 C CNN
-F 3 "" H 4150 3850 50  0001 C CNN
-	1    4150 3850
+F 0 "#PWR0138" H 4250 3950 50  0001 C CNN
+F 1 "-5V" H 4265 4023 50  0000 C CNN
+F 2 "" H 4250 3850 50  0001 C CNN
+F 3 "" H 4250 3850 50  0001 C CNN
+	1    4250 3850
 	-1   0    0    1
 $EndComp
 Wire Wire Line
-	3900 3150 4250 3150
-Wire Wire Line
-	4250 3150 4250 3350
+	3900 3150 4150 3150
 $Comp
 L Device:R_Small R?
@@
 L Device:C_Small C?
 U 1 1 5BDB24A8
-P 4600 3800
+P 4700 3800
 AR Path="/5BCA1695/5BDB24A8" Ref="C?"  Part="1"
 AR Path="/5BE0B501/5BDB24A8" Ref="C?"  Part="1"
 AR Path="/5BDB24A8" Ref="C?"  Part="1"
 AR Path="/5BD77D91/5BDB24A8" Ref="C5"  Part="1"
-F 0 "C5" V 4371 3800 50  0000 R CNN
-F 1 "0603B104M500CT " V 4462 3800 50  0000 C CNN
-F 2 "Resistor_SMD:R_0603_1608Metric" H 4600 3800 50  0001 C CNN
-F 3 "http://www.passivecomponent.com/indexsea/ASC_General_Purpose.pdf" H 4600 3800 50  0001 C CNN
-	1    4600 3800
-	0    -1   -1   0
-$EndComp
-Wire Wire Line
-	4700 3800 4800 3800
+F 0 "C5" V 4471 3800 50  0000 R CNN
+F 1 "0603B104M500CT " V 4562 3800 50  0000 C CNN
+F 2 "Resistor_SMD:R_0603_1608Metric" H 4700 3800 50  0001 C CNN
+F 3 "http://www.passivecomponent.com/indexsea/ASC_General_Purpose.pdf" H 4700 3800 50  0001 C CNN
+	1    4700 3800
+	0    -1   -1   0
+$EndComp
+Wire Wire Line
+	4800 3800 4900 3800
 $Comp
 L power:GND #PWR?
 U 1 1 5BDB24AF
-P 4800 3800
+P 4900 3800
 AR Path="/5BCA1695/5BDB24AF" Ref="#PWR?"  Part="1"
 AR Path="/5BE0B501/5BDB24AF" Ref="#PWR?"  Part="1"
 AR Path="/5BDB24AF" Ref="#PWR?"  Part="1"
 AR Path="/5BD77D91/5BDB24AF" Ref="#PWR0140"  Part="1"
-F 0 "#PWR0140" H 4800 3550 50  0001 C CNN
-F 1 "GND" V 4805 3672 50  0000 R CNN
-F 2 "" H 4800 3800 50  0001 C CNN
-F 3 "" H 4800 3800 50  0001 C CNN
-	1    4800 3800
+F 0 "#PWR0140" H 4900 3550 50  0001 C CNN
+F 1 "GND" V 4905 3672 50  0000 R CNN
+F 2 "" H 4900 3800 50  0001 C CNN
+F 3 "" H 4900 3800 50  0001 C CNN
+	1    4900 3800
 	0    -1   -1   0
 $EndComp
@@
 	4150 2400 4150 2600
 Wire Wire Line
-	4150 3800 4500 3800
-Connection ~ 4150 3800
-Wire Wire Line
-	4150 3800 4150 3850
+	4250 3800 4600 3800
+Connection ~ 4250 3800
+Wire Wire Line
+	4250 3800 4250 3850
 Wire Wire Line
 	5450 4400 5450 4650
@@
 Wire Wire Line
 	5550 4400 5550 4950
+Connection ~ 4150 3150
+Wire Wire Line
+	4150 3150 4250 3150
+Wire Wire Line
+	4150 3150 4150 3300
+NoConn ~ 4150 3650
 $EndSCHEMATC
