File: pcb/pro/Ntester/InAmp.sch (KiCad schematic (older format))
At the start: 23 parts, among them Q1 BC847BDW1T1G, U1 LT1818

Commit message: layout finalized
Parts:
- removed TP1, TP4: TestPoint, TestPoint:TestPoint_THTPad_D1.0mm_Drill0.5mm, symbol Connector:TestPoint
Connections:
- net at C9.1, R1.2, TP5.1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: now also C12.2, C13.2, C14.2; no longer C12.1, C13.1, C14.1
- new net: C12.1, C13.1, C14.1, R6.2
Other:
- moved on the sheet: C12, C14

Commit message: BOM was updated
Connections:
- net IN_AMP: no longer RN1.2 (R2.1), RN1.7 (R2.2)
- new net: RN1.2 (R2.1), RN1.7 (R2.2)
Changed lines of the file:
@@
 $EndComp
 Wire Wire Line
-	5100 4750 5100 5900
-Wire Wire Line
 	5100 4350 5100 4750
-Connection ~ 5100 4750
 $Comp
 L Device:R_Pack04 RN1
