File: pcb/pro/Ntester/LNA3.sch (KiCad schematic (older format))
At the start: 21 parts, among them Q4 BC847BDW1T1G, U7 LT1818

Commit message: BOM was updated
Connections:
- net IN_AMP: no longer RN4.2 (R2.1), RN4.7 (R2.2)
- new net: RN4.2 (R2.1), RN4.7 (R2.2)
Changed lines of the file:
@@
 	4599 4022 4599 4422
-Wire Wire Line
-	4599 4422 4599 5572
 Wire Wire Line
 	4599 5572 2499 5572
 Wire Wire Line
 	2499 5572 2499 3472
-Connection ~ 4599 4422
 Connection ~ 2499 3472
 Wire Wire Line
