File: pcb/pro/Ntester/Ntester.kicad_pcb (KiCad board)
At the start: 4 copper layers, 102 parts, among them J1 Conn_Coaxial, J2 Conn_01x02_Male, J3 RF_Shield_One_Piece, J4 67996-408HLF, J5 Conn_Coaxial, J6 Conn_Coaxial, Q1 BC847BDW1T1G, U1 LT1818

Commit message: " alomost" finalized layout
Parts:
- removed the C1 at (68.1, 143.7)
- removed the C1 at (68.3, 132.6)
- removed the C1 at (68.2, 121.3)
- removed the C10 at (76.3, 128.4)
- removed the C10 at (76.1, 139.5)
- removed the C10 at (76.2, 117.1)
- removed the C11 at (74.0, 142.0)
- removed the C11 at (74.2, 130.9)
- removed the C11 at (74.1, 119.7)
- removed the C12 at (83.1, 139.6)
- removed the C12 at (83.3, 128.4)
- removed the C12 at (83.2, 117.2)
- removed the C13 at (83.1, 144.5)
- removed the C13 at (83.3, 133.3)
- removed the C13 at (83.2, 122.1)
- removed the C13 at (83.4, 111.0)
- removed the C14 at (82.9, 143.4)
- removed the C14 at (83.1, 132.2)
- removed the C14 at (83.0, 121.0)
- removed the C15 at (63.0, 131.7)
- removed the C15 at (62.8, 142.9)
- removed the C15 at (62.9, 120.5)
- removed the C16 at (63.0, 128.6)
- removed the C16 at (62.7, 139.7)
- removed the C16 at (62.8, 117.3)
- removed the C3 at (68.2, 127.7)
- removed the C3 at (68.0, 138.8)
- removed the C3 at (68.1, 116.4)
- removed the C8 at (69.4, 141.7)
- removed the C8 at (69.6, 130.6)
- removed the C8 at (69.5, 119.3)
- removed the C9 at (72.8, 138.3)
- removed the C9 at (73.0, 127.2)
- removed the C9 at (72.9, 115.9)
- removed the Q1 at (69.5, 143.8)
- removed the Q1 at (69.7, 132.7)
- removed the Q1 at (69.6, 121.4)
- removed the Q1 at (69.8, 110.3)
- removed the R1 at (76.2, 143.7)
- removed the R1 at (76.4, 132.6)
- removed the R1 at (76.3, 121.3)
- removed the R2 at (73.2, 143.7)
- removed the R2 at (73.4, 132.6)
- removed the R2 at (73.3, 121.3)
- removed the R4 at (69.5, 127.5)
- removed the R4 at (69.3, 138.6)
- removed the R4 at (69.4, 116.2)
- removed the R5 at (69.5, 140.2)
- removed the R5 at (69.7, 129.1)
- removed the R5 at (69.6, 117.8)
- removed REF**: Wuerth_36503505_50x50mm, RF_Shielding:Wuerth_36503505_50x50mm
- removed the RN1 at (65.5, 129.6)
- removed the RN1 at (65.3, 140.7)
- removed the RN1 at (65.4, 118.3)
- removed the U1 at (74.5, 141.0)
- removed the U1 at (74.7, 129.9)
- removed the U1 at (74.6, 118.6)
- added C13: B45196-H2227-M409, Capacitor_Tantalum_SMD:CP_EIA-7343-31_Kemet-D, F.Cu at (88.5, 106.5)
- added C17: DNP, Capacitor_SMD:C_0603_1608Metric, F.Cu at (104.4, 125.7)
- added C26: 0603B104M500CT, Resistor_SMD:R_0603_1608Metric, F.Cu at (104.5, 141.3)
- added C27: 0603B104M500CT, Resistor_SMD:R_0603_1608Metric, F.Cu at (109.4, 133.2)
- added C28: B45196-H2227-M409, Capacitor_Tantalum_SMD:CP_EIA-7343-31_Kemet-D, B.Cu at (108.0, 134.8)
- added C29: SMDTD04470YA00MT00, Ntester:CAP-6054-SMDTD04470YA00MT00, B.Cu at (112.0, 110.9)
- added C30: C_Small, Capacitor_SMD:C_0603_1608Metric, F.Cu at (102.0, 138.6)
- added C31: C_Small, Capacitor_SMD:C_0603_1608Metric, F.Cu at (102.0, 136.8)
- added C32: DNP, Capacitor_SMD:C_0603_1608Metric, F.Cu at (113.3, 138.5)
- added C33: C_Small, Capacitor_SMD:C_0603_1608Metric, F.Cu at (107.2, 144.8)
- added C34: C_Small, Capacitor_SMD:C_0603_1608Metric, F.Cu at (104.0, 147.9)
- added C35: B45196-H2227-M409, Capacitor_Tantalum_SMD:CP_EIA-7343-31_Kemet-D, F.Cu at (88.7, 159.7)
- added C36: B45196-H2227-M409, Capacitor_Tantalum_SMD:CP_EIA-7343-31_Kemet-D, F.Cu at (93.6, 159.7)
- added C37: B45196-H2227-M409, Capacitor_Tantalum_SMD:CP_EIA-7343-31_Kemet-D, F.Cu at (110.3, 159.6)
- added C38: B45196-H2227-M409, Capacitor_Tantalum_SMD:CP_EIA-7343-31_Kemet-D, F.Cu at (115.3, 159.6)
- added C39: B45196-H2227-M409, Capacitor_Tantalum_SMD:CP_EIA-7343-31_Kemet-D, B.Cu at (109.5, 147.2)
- added C40: 0603B104M500CT, Resistor_SMD:R_0603_1608Metric, F.Cu at (114.8, 145.9)
- added C41: 0603B104M500CT, Resistor_SMD:R_0603_1608Metric, F.Cu at (107.3, 152.3)
- added C42: B45196-H2227-M409, Capacitor_Tantalum_SMD:CP_EIA-7343-31_Kemet-D, B.Cu at (109.5, 152.1)
- added C43: 885012006007, Resistor_SMD:R_0603_1608Metric, F.Cu at (56.7, 161.2)
- added C44: 885012006007, Resistor_SMD:R_0603_1608Metric, F.Cu at (65.0, 161.2)
- added D3: BAS116LT1G, Package_TO_SOT_SMD:SOT-23, F.Cu at (53.7, 161.0)
- added D4: BAS116LT1G, Package_TO_SOT_SMD:SOT-23, F.Cu at (68.2, 161.0)
- added D5: LED_Small, Resistor_SMD:R_0805_2012Metric, F.Cu at (68.2, 154.9)
- added F1: Polyfuse_Small, Resistor_SMD:R_0805_2012Metric, F.Cu at (54.6, 165.2)
- added F2: Polyfuse_Small, Resistor_SMD:R_0805_2012Metric, F.Cu at (67.3, 165.3)
- added H1: M3.5, MountingHole:MountingHole_3.5mm_Pad_Via, F.Cu at (121.8, 96.2)
- added H2: M3.5, MountingHole:MountingHole_3.5mm_Pad_Via, F.Cu at (121.8, 163.8)
- added H3: M3.5, MountingHole:MountingHole_3.5mm_Pad_Via, F.Cu at (30.2, 96.2)
- added H4: M3.5, MountingHole:MountingHole_3.5mm_Pad_Via, F.Cu at (30.2, 163.8)
- added J7: 36503505S 36003500S, RF_Shielding:Wuerth_36503505_50x50mm, F.Cu at (72.8, 121.2)
- added J8: PWR IN, Connector_PinHeader_2.54mm:PinHeader_1x03_P2.54mm_Vertical, F.Cu at (58.5, 165.3)
- added JP2: GND_SHIELD, Jumper:SolderJumper-2_P1.3mm_Open_TrianglePad1.0x1.5mm, F.Cu at (115.6, 96.2)
- added JP3: GND_SHIELD, Jumper:SolderJumper-2_P1.3mm_Open_TrianglePad1.0x1.5mm, F.Cu at (121.9, 157.6)
- added JP4: GND_SHIELD, Jumper:SolderJumper-2_P1.3mm_Open_TrianglePad1.0x1.5mm, F.Cu at (36.4, 96.2)
- added JP5: GND_SHIELD, Jumper:SolderJumper-2_P1.3mm_Open_TrianglePad1.0x1.5mm, F.Cu at (28.6, 157.9)
- added Q1: BC847BDW1T1G, Package_TO_SOT_SMD:SOT-363_SC-70-6, F.Cu at (71.1, 106.7)
- added R11: R_Small, Resistor_SMD:R_0603_1608Metric, F.Cu at (116.2, 126.4)
- added R12: R_Small, Resistor_SMD:R_0603_1608Metric, F.Cu at (116.2, 129.0)
- added R13: R_Small, Resistor_SMD:R_0603_1608Metric, F.Cu at (102.0, 133.5)
- added R14: R_Small, Resistor_SMD:R_0603_1608Metric, F.Cu at (114.9, 138.5)
- added R15: R_Small, Resistor_SMD:R_0603_1608Metric, F.Cu at (102.0, 135.0)
- added R16: R_Small, Resistor_SMD:R_0603_1608Metric, F.Cu at (114.1, 136.0)
- added R17: R_Small, Resistor_SMD:R_0603_1608Metric, F.Cu at (114.1, 141.0)
- added R18: R_Small, Resistor_SMD:R_0603_1608Metric, F.Cu at (105.6, 143.2)
- added R19: R_Small, Resistor_SMD:R_0603_1608Metric, F.Cu at (104.8, 145.6)
- added R20: R_Small, Resistor_SMD:R_1206_3216Metric, F.Cu at (88.6, 165.4)
- added R21: R_Small, Resistor_SMD:R_1206_3216Metric, F.Cu at (110.2, 165.4)
- added R22: 10k, Resistor_SMD:R_0805_2012Metric, F.Cu at (65.5, 154.9)
- added SW1: JS202011CQN, Button_Switch_THT:SW_CuK_JS202011CQN_DPDT_Straight, F.Cu at (59.2, 160.8)
- added TP1: TestPoint, TestPoint:TestPoint_THTPad_D1.0mm_Drill0.5mm, F.Cu at (58.8, 100.4)
- added TP10: TestPoint, TestPoint:TestPoint_THTPad_D1.0mm_Drill0.5mm, F.Cu at (111.0, 143.9)
- added TP11: TestPoint, TestPoint:TestPoint_THTPad_D1.0mm_Drill0.5mm, F.Cu at (62.5, 151.6)
- added TP12: TestPoint, TestPoint:TestPoint_THTPad_D1.0mm_Drill0.5mm, F.Cu at (58.0, 149.6)
- added TP2: TestPoint, TestPoint:TestPoint_THTPad_D1.0mm_Drill0.5mm, F.Cu at (53.0, 158.0)
- added TP3: TestPoint, TestPoint:TestPoint_THTPad_D1.0mm_Drill0.5mm, F.Cu at (75.6, 107.1)
- added TP4: TestPoint, TestPoint:TestPoint_THTPad_D1.0mm_Drill0.5mm, F.Cu at (52.2, 100.4)
- added TP5: TestPoint, TestPoint:TestPoint_THTPad_D1.0mm_Drill0.5mm, F.Cu at (82.5, 107.1)
- added TP6: TestPoint, TestPoint:TestPoint_THTPad_D1.0mm_Drill0.5mm, F.Cu at (56.8, 158.3)
- added TP7: TestPoint, TestPoint:TestPoint_THTPad_D1.0mm_Drill0.5mm, F.Cu at (65.4, 158.3)
- added TP8: TestPoint, TestPoint:TestPoint_THTPad_D1.0mm_Drill0.5mm, F.Cu at (102.3, 123.1)
- added TP9: TestPoint, TestPoint:TestPoint_THTPad_D1.0mm_Drill0.5mm, F.Cu at (113.8, 133.9)
- added U2: LT6231, Ntester:SOIC-8-LINEAR, F.Cu at (109.9, 127.1)
- added U3: LT6231, Ntester:SOIC-8-LINEAR, F.Cu at (108.3, 137.1)
- added U4: LT1364, Ntester:SOIC-8-LINEAR, F.Cu at (109.9, 148.6)
- C18, C19: moved to B.Cu
- C2: value B45196-H2227-M409 -> 885012006007; footprint Capacitor_Tantalum_SMD:CP_EIA-7343-31_Kemet-D -> Resistor_SMD:R_0603_1608Metric
- C22: value 0603B104M500CT -> B45196-H2227-M409; footprint Resistor_SMD:R_0603_1608Metric -> Capacitor_Tantalum_SMD:CP_EIA-7343-31_Kemet-D
- C23: value 0603B104M500CT -> DNP; footprint Resistor_SMD:R_0603_1608Metric -> Capacitor_Tantalum_SMD:CP_EIA-7343-31_Kemet-D
- C24: value ECW-FE2W475J -> SMDTD04470YA00MT00; footprint Capacitor_THT:C_Rect_L26.5mm_W11.5mm_P22.50mm_MKS4 -> Ntester:CAP-6054-SMDTD04470YA00MT00
- C25: value 16MU475MC14532 -> B45196-H2227-M409; footprint Capacitor_SMD:C_1812_4532Metric -> Capacitor_Tantalum_SMD:CP_EIA-7343-31_Kemet-D; moved to B.Cu
- C4: value 885012006007 -> 0603B104M500CT
- C5: value B45196-H2227-M409 -> 0603B104M500CT; footprint Capacitor_Tantalum_SMD:CP_EIA-7343-31_Kemet-D -> Resistor_SMD:R_0603_1608Metric
- C7: value DNP -> B45196-H2227-M409
- J1: value Conn_Coaxial -> Conn_01x02_Male; footprint Connector_Coaxial:BNC_TEConnectivity_1478204_Vertical -> Connector_PinHeader_2.54mm:PinHeader_1x02_P2.54mm_Vertical
- J2: value Conn_01x02_Male -> Conn_Coaxial; footprint Connector_PinHeader_2.54mm:PinHeader_1x02_P2.54mm_Vertical -> Connector_Coaxial:BNC_TEConnectivity_1478204_Vertical
- J3: value RF_Shield_One_Piece -> Conn_Coaxial; footprint RF_Shielding:Wuerth_36103205_20x20mm -> Connector_Coaxial:BNC_TEConnectivity_1478204_Vertical
- R10: value RMCF0603FT499R -> RMCF0603FT499R
- R3: value RMCF0603FT499R -> RHC2512FT4R99; footprint Resistor_SMD:R_0603_1608Metric -> Resistor_SMD:R_2512_6332Metric
- R7: value RHC2512FT4R99 -> CRM2512-JW-470ELF
- R8: value CRM2512-JW-470ELF -> CR1206-FX-4990ELF; footprint Resistor_SMD:R_2512_6332Metric -> Resistor_SMD:R_1206_3216Metric
- R9: value CR1206-FX-4990ELF -> RMCF0603FT499R; footprint Resistor_SMD:R_1206_3216Metric -> Resistor_SMD:R_0603_1608Metric
- U1: footprint Package_SO:MSOP-8_3x3mm_P0.65mm -> Ntester:SOIC-8-LINEAR
- moved D2 124.0 mm to (43.6, 143.2)
- moved D1 119.8 mm to (43.6, 139.4), turned to 90 degrees
- moved C22 116.0 mm to (56.0, 110.0)
- moved J5 116.0 mm to (80.5, 161.0), turned to 270 degrees
- moved C23 115.7 mm to (56.0, 122.0)
- moved J6 99.5 mm to (102.1, 161.0), turned to 270 degrees
- moved J3 69.3 mm to (33.0, 107.0), turned to 90 degrees
- moved C5 42.8 mm to (43.4, 146.2), turned to 180 degrees
- moved R10 38.9 mm to (102.3, 125.7), turned to 90 degrees
- moved R6 32.6 mm to (91.4, 109.8)
- moved C20 32.6 mm to (107.9, 131.0)
- moved JP1 32.0 mm to (28.2, 145.5), turned to 90 degrees
- moved R3 30.6 mm to (31.1, 137.6)
- moved R9 29.0 mm to (56.0, 100.4), turned to 180 degrees
- moved C25 28.9 mm to (108.0, 139.7)
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Connections:
- net /InputStage/R_LTP0 renamed /InputAmplifier/R_LTP0
- net /InputStage/R_LTP2 renamed /InputAmplifier/R_LTP2
- C2 pad 2: /InputStage/IN_SIG -> GND
- C20 pad 1: GND -> -5V
- C20 pad 2: -5V -> GND
- C22 pad 1: +5V -> Net-(C2-Pad1)
- C22 pad 2: GND -> /InputAmplifier/IN_AMP
- C23 pad 1: +5V -> Net-(C2-Pad1)
- C23 pad 2: GND -> /InputAmplifier/IN_AMP
- C24 pad 2: Net-(C24-Pad2) -> Net-(C17-Pad1)
- C25 pad 1: Net-(C25-Pad1) -> +5V
- C25 pad 2: Net-(C25-Pad2) -> GND
- C4 pad 1: Net-(C2-Pad1) -> +5V
- C5 pad 1: Net-(C2-Pad1) -> -5V
- C5 pad 2: /InputStage/IN_SIG -> GND
- C6 pad 2: /InputStage/IN_SIG -> /InputAmplifier/IN_AMP
- C7 pad 2: /InputStage/IN_SIG -> /InputAmplifier/IN_AMP
- D1 pad 2: Net-(D1-Pad2) -> (no net)
- D2 pad 2: Net-(D2-Pad2) -> (no net)
- FB1 pad 2: Net-(FB1-Pad2) -> /InputStage/IN_STG
- J1 pad 1: Net-(FB1-Pad2) -> /InputStage/IN_STG
- J2 pad 1: Net-(FB1-Pad2) -> /InputStage/IN_STG
- J3 pad 1: Net-(J3-Pad1) -> /InputStage/IN_STG
- J5 pad 1: Net-(J5-Pad1) -> /GainBlock/WB_OUT
- J6 pad 1: Net-(J6-Pad1) -> /GainBlock/1MHZ_OUT
- JP1 pad 1: Net-(J4-Pad8) -> Net-(J4-Pad2)
- R10 pad 2: Net-(R10-Pad2) -> Net-(C17-Pad1)
- R3 pad 1: /InputStage/IN_SIG -> Net-(J4-Pad8)
- R6 pad 1: /InputStage/OUT_SIG -> /GainBlock/GB_IN
- R9 pad 1: Net-(J4-Pad2) -> /InputAmplifier/IN_AMP
- RN1 pad 1: /InputStage/R_LTP5 -> /InputAmplifier/R_LTP5
- RN1 pad 2: /InputStage/IN_SIG -> /InputAmplifier/IN_AMP
- RN1 pad 7: /InputStage/IN_SIG -> /InputAmplifier/IN_AMP
- U1 pad 1: Net-(U1-Pad1) -> (no net)
- U1 pad 5: Net-(U1-Pad5) -> (no net)
- U1 pad 8: Net-(U1-Pad8) -> (no net)
Routing:
- net +5V: track 13.9 -> 247.3 mm, vias 4 -> 11
- net -5V: track 10.8 -> 216.5 mm, vias 4 -> 10
- net Net-(C2-Pad1): track 0.00 -> 63.8 mm
- net GND: track 0.00 -> 51.2 mm, vias 0 -> 75
- net /InputStage/IN_SIG: track 46.0 -> 0.00 mm
- net Net-(C12-Pad1): track 70.2 -> 25.5 mm
- net Net-(C29-Pad1): track 0.00 -> 31.9 mm, vias 0 -> 2
- net /GainBlock/GB_IN: track 0.00 -> 31.7 mm
- net /InputStage/R_LTP5: track 30.6 -> 0.00 mm
- net /InputStage/IN_STG: track 0.00 -> 29.4 mm
- net Net-(C33-Pad1): track 0.00 -> 29.3 mm
- net Net-(C32-Pad1): track 0.00 -> 27.1 mm
- net /InputAmplifier/R_LTP0: track 32.4 -> 7.04 mm
- net /InputAmplifier/R_LTP2: track 32.0 -> 7.98 mm
- net Net-(C17-Pad1): track 0.00 -> 20.3 mm
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- added copper zone on B.Cu, net GND
- added copper zone on F.Cu, net GND
- added copper zone on In1.Cu, net GND
Other:
- board outline added: 100 x 76 mm
- net class PWR added: clearance 0.3, trace_width 0.35, via_dia 0.8, via_drill 0.4
- net class thicc added: clearance 0.2, trace_width 0.4, via_dia 0.8, via_drill 0.4
- board text added: "1MHz OUT"
- board text added: "POLARIZATION OF TANTALUM CAPS"
- board text added: "WB OUT"

Commit message: layout finalized
Parts:
- added C45: GRM32ER60J107ME20K, Capacitor_SMD:C_1210_3225Metric, B.Cu at (110.9, 157.4)
- added C46: GRM32ER60J107ME20K, Capacitor_SMD:C_1210_3225Metric, F.Cu at (119.2, 157.4)
- added C47: GRM32ER60J107ME20K, Capacitor_SMD:C_1210_3225Metric, B.Cu at (115.0, 157.4)
- added C48: GRM32ER60J107ME20K, Capacitor_SMD:C_1210_3225Metric, F.Cu at (89.3, 160.7)
- added C49: GRM32ER60J107ME20K, Capacitor_SMD:C_1210_3225Metric, B.Cu at (89.3, 164.9)
- added C50: GRM32ER60J107ME20K, Capacitor_SMD:C_1210_3225Metric, F.Cu at (89.3, 164.9)
- added C51: GRM32ER60J107ME20K, Capacitor_SMD:C_1210_3225Metric, B.Cu at (89.3, 160.7)
- added C52: GRM32ER60J107ME20K, Capacitor_SMD:C_1210_3225Metric, F.Cu at (89.3, 152.2)
- added C53: GRM32ER60J107ME20K, Capacitor_SMD:C_1210_3225Metric, B.Cu at (89.3, 156.5)
- added C54: GRM32ER60J107ME20K, Capacitor_SMD:C_1210_3225Metric, F.Cu at (89.3, 156.4)
- added C55: 885012006038, Resistor_SMD:R_0603_1608Metric, F.Cu at (71.0, 115.8)
- added C56: 0603B104M500CT, Resistor_SMD:R_0603_1608Metric, B.Cu at (79.5, 112.6)
- added C57: 885012006007, Resistor_SMD:R_0603_1608Metric, F.Cu at (74.0, 112.8)
- added C58: 0603B104M500CT, Resistor_SMD:R_0603_1608Metric, B.Cu at (79.5, 115.8)
- added C59: B45196-H2227-M409, Capacitor_Tantalum_SMD:CP_EIA-7343-31_Kemet-D, B.Cu at (70.0, 118.0)
- added C60: DNP, Capacitor_Tantalum_SMD:CP_EIA-7343-31_Kemet-D, F.Cu at (88.5, 118.0)
- added C61: B45196-H2227-M409, Capacitor_Tantalum_SMD:CP_EIA-7343-31_Kemet-D, F.Cu at (88.5, 113.1)
- added C62: B45196-H2227-M409, Capacitor_Tantalum_SMD:CP_EIA-7343-31_Kemet-D, B.Cu at (88.5, 113.1)
- added C63: B45196-H2227-M409, Capacitor_Tantalum_SMD:CP_EIA-7343-31_Kemet-D, B.Cu at (70.0, 113.1)
- added C64: 0603B104M500CT, Resistor_SMD:R_0603_1608Metric, B.Cu at (64.7, 117.1)
- added C65: 0603B104M500CT, Resistor_SMD:R_0603_1608Metric, B.Cu at (64.7, 114.0)
- added C66: 885012006038, Resistor_SMD:R_0603_1608Metric, F.Cu at (71.0, 127.3)
- added C67: 0603B104M500CT, Resistor_SMD:R_0603_1608Metric, B.Cu at (79.5, 124.0)
- added C68: 885012006007, Resistor_SMD:R_0603_1608Metric, F.Cu at (74.0, 124.3)
- added C69: 0603B104M500CT, Resistor_SMD:R_0603_1608Metric, B.Cu at (79.5, 127.5)
- added C70: B45196-H2227-M409, Capacitor_Tantalum_SMD:CP_EIA-7343-31_Kemet-D, B.Cu at (70.0, 129.5)
- added C71: DNP, Capacitor_Tantalum_SMD:CP_EIA-7343-31_Kemet-D, B.Cu at (88.5, 124.6)
- added C72: B45196-H2227-M409, Capacitor_Tantalum_SMD:CP_EIA-7343-31_Kemet-D, F.Cu at (88.5, 129.5)
- added C73: B45196-H2227-M409, Capacitor_Tantalum_SMD:CP_EIA-7343-31_Kemet-D, F.Cu at (88.5, 124.6)
- added C74: B45196-H2227-M409, Capacitor_Tantalum_SMD:CP_EIA-7343-31_Kemet-D, B.Cu at (70.0, 124.6)
- added C75: 0603B104M500CT, Resistor_SMD:R_0603_1608Metric, B.Cu at (64.7, 128.6)
- added C76: 0603B104M500CT, Resistor_SMD:R_0603_1608Metric, B.Cu at (64.7, 125.5)
- added C77: 885012006038, Resistor_SMD:R_0603_1608Metric, F.Cu at (71.0, 138.8)
- added C78: 0603B104M500CT, Resistor_SMD:R_0603_1608Metric, B.Cu at (79.5, 135.5)
- added C79: 885012006007, Resistor_SMD:R_0603_1608Metric, F.Cu at (74.0, 135.8)
- added C80: 0603B104M500CT, Resistor_SMD:R_0603_1608Metric, B.Cu at (79.5, 139.0)
- added C81: B45196-H2227-M409, Capacitor_Tantalum_SMD:CP_EIA-7343-31_Kemet-D, B.Cu at (70.0, 141.0)
- added C82: DNP, Capacitor_Tantalum_SMD:CP_EIA-7343-31_Kemet-D, B.Cu at (88.5, 136.1)
- added C83: B45196-H2227-M409, Capacitor_Tantalum_SMD:CP_EIA-7343-31_Kemet-D, F.Cu at (88.5, 136.1)
- added C84: B45196-H2227-M409, Capacitor_Tantalum_SMD:CP_EIA-7343-31_Kemet-D, F.Cu at (88.5, 141.0)
- added C85: B45196-H2227-M409, Capacitor_Tantalum_SMD:CP_EIA-7343-31_Kemet-D, B.Cu at (70.0, 136.1)
- added C86: 0603B104M500CT, Resistor_SMD:R_0603_1608Metric, B.Cu at (64.7, 140.1)
- added C87: 0603B104M500CT, Resistor_SMD:R_0603_1608Metric, B.Cu at (64.7, 137.0)
- added Q2: BC847BDW1T1G, Package_TO_SOT_SMD:SOT-363_SC-70-6, F.Cu at (71.1, 118.2)
- added Q3: BC847BDW1T1G, Package_TO_SOT_SMD:SOT-363_SC-70-6, F.Cu at (71.1, 129.7)
- added Q4: BC847BDW1T1G, Package_TO_SOT_SMD:SOT-363_SC-70-6, F.Cu at (71.1, 141.2)
- added R23: CR0603-JW-471ELF, Resistor_SMD:R_0603_1608Metric, F.Cu at (71.0, 112.8)
- added R24: CR0603-JW-471ELF, Resistor_SMD:R_0603_1608Metric, F.Cu at (71.0, 114.3)
- added R25: RNCF0603TKY250R, Resistor_SMD:R_0603_1608Metric, F.Cu at (78.4, 118.6)
- added R26: RNCF0603AKT10R0, Resistor_SMD:R_0603_1608Metric, F.Cu at (73.7, 117.4)
- added R27: RG1608N-101-W-T1, Resistor_SMD:R_0603_1608Metric, F.Cu at (94.6, 115.5)
- added R28: CR0603-JW-471ELF, Resistor_SMD:R_0603_1608Metric, F.Cu at (71.0, 124.3)
- added R29: CR0603-JW-471ELF, Resistor_SMD:R_0603_1608Metric, F.Cu at (71.0, 125.8)
- added R30: RNCF0603TKY250R, Resistor_SMD:R_0603_1608Metric, F.Cu at (78.4, 130.1)
- added R31: RNCF0603AKT10R0, Resistor_SMD:R_0603_1608Metric, F.Cu at (73.7, 128.9)
- added R32: RG1608N-101-W-T1, Resistor_SMD:R_0603_1608Metric, F.Cu at (94.6, 127.0)
- added R33: CR0603-JW-471ELF, Resistor_SMD:R_0603_1608Metric, F.Cu at (71.0, 135.8)
- added R34: CR0603-JW-471ELF, Resistor_SMD:R_0603_1608Metric, F.Cu at (71.0, 137.3)
- added R35: RNCF0603TKY250R, Resistor_SMD:R_0603_1608Metric, F.Cu at (78.4, 141.6)
- added R36: RNCF0603AKT10R0, Resistor_SMD:R_0603_1608Metric, F.Cu at (73.7, 140.4)
- added R37: RG1608N-101-W-T1, Resistor_SMD:R_0603_1608Metric, F.Cu at (94.6, 138.5)
- added REF**: OSHW-Logo2_7.3x6mm_SilkScreen, Symbol:OSHW-Logo2_7.3x6mm_SilkScreen, F.Cu at (105.4, 97.0)
- added RN2: ACASA1001S1001P1AT, Resistor_SMD:R_Array_Convex_4x1206, F.Cu at (67.0, 114.9)
- added RN3: ACASA1001S1001P1AT, Resistor_SMD:R_Array_Convex_4x1206, F.Cu at (67.0, 126.4)
- added RN4: ACASA1001S1001P1AT, Resistor_SMD:R_Array_Convex_4x1206, F.Cu at (67.0, 137.9)
- added TP13: TestPoint, TestPoint:TestPoint_THTPad_D1.0mm_Drill0.5mm, F.Cu at (75.6, 130.1)
- added TP14: TestPoint, TestPoint:TestPoint_THTPad_D1.0mm_Drill0.5mm, F.Cu at (75.6, 118.6)
- added TP15: TestPoint, TestPoint:TestPoint_THTPad_D1.0mm_Drill0.5mm, F.Cu at (82.5, 130.1)
- added TP16: TestPoint, TestPoint:TestPoint_THTPad_D1.0mm_Drill0.5mm, F.Cu at (82.5, 118.6)
- added TP17: TestPoint, TestPoint:TestPoint_THTPad_D1.0mm_Drill0.5mm, F.Cu at (75.6, 141.6)
- added TP18: TestPoint, TestPoint:TestPoint_THTPad_D1.0mm_Drill0.5mm, F.Cu at (82.5, 141.6)
- added U5: LT1818, Ntester:SOIC-8-LINEAR, F.Cu at (79.6, 114.4)
- added U6: LT1818, Ntester:SOIC-8-LINEAR, F.Cu at (79.6, 125.9)
- added U7: LT1818, Ntester:SOIC-8-LINEAR, F.Cu at (79.6, 137.4)
- C35, C36, C38: value B45196-H2227-M409 -> GRM32ER60J107ME20K; footprint Capacitor_Tantalum_SMD:CP_EIA-7343-31_Kemet-D -> Capacitor_SMD:C_1210_3225Metric
- C37: value B45196-H2227-M409 -> GRM32ER60J107ME20K; footprint Capacitor_Tantalum_SMD:CP_EIA-7343-31_Kemet-D -> Capacitor_SMD:C_1210_3225Metric; moved to B.Cu
- J8: footprint Connector_PinHeader_2.54mm:PinHeader_1x03_P2.54mm_Vertical -> Connector_PinHeader_2.54mm:PinHeader_1x04_P2.54mm_Vertical
- moved C35 26.5 mm to (115.1, 157.4), turned to 90 degrees
- moved C36 17.5 mm to (110.9, 157.4), turned to 90 degrees
- moved R20 12.3 mm to (83.8, 154.1)
- moved C38 8.80 mm to (106.8, 157.4), turned to 90 degrees
- moved R6 6.62 mm to (94.6, 104.0)
- moved C34 5.55 mm to (108.6, 144.8), turned to 0 degrees
- moved R21 4.33 mm to (106.8, 162.7), turned to 270 degrees
- moved C37 4.14 mm to (106.8, 157.4), turned to 90 degrees
- moved C33 3.47 mm to (104.7, 147.2), turned to 90 degrees
- moved J6 2.82 mm to (99.3, 161.3)
- moved J8 1.92 mm to (56.6, 165.0)
- moved JP3 1.80 mm to (123.7, 157.5)
- moved F1 1.08 mm to (53.6, 164.8), turned to 270 degrees
- moved R19 1.06 mm to (105.5, 144.8), turned to 0 degrees
- moved F2 0.86 mm to (68.0, 164.8), turned to 270 degrees
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Connections:
- C35 pad 1: Net-(C33-Pad1) -> /GainBlock/1MHZ_OUT
- C35 pad 2: /GainBlock/WB_OUT -> Net-(C35-Pad2)
- C36 pad 1: Net-(C33-Pad1) -> /GainBlock/1MHZ_OUT
- C36 pad 2: /GainBlock/WB_OUT -> Net-(C35-Pad2)
- C37 pad 1: Net-(C37-Pad1) -> /GainBlock/1MHZ_OUT
- C37 pad 2: /GainBlock/1MHZ_OUT -> Net-(C35-Pad2)
- C38 pad 1: Net-(C37-Pad1) -> /GainBlock/1MHZ_OUT
- C38 pad 2: /GainBlock/1MHZ_OUT -> Net-(C35-Pad2)
- C9 pad 1: Net-(C12-Pad1) -> Net-(C12-Pad2)
- D2 pad 1: Net-(C2-Pad1) -> -5V
- D2 pad 3: -5V -> Net-(C2-Pad1)
- D4 pad 1: GND -> Net-(C44-Pad1)
- D4 pad 3: Net-(C44-Pad1) -> GND
- J8 pad 3: Net-(F2-Pad2) -> GND
- R1 pad 2: Net-(C12-Pad1) -> Net-(C12-Pad2)
- R6 pad 2: Net-(C12-Pad2) -> Net-(C12-Pad1)
- TP5 pad 1: Net-(C12-Pad1) -> Net-(C12-Pad2)
- U1 pad 6: Net-(C12-Pad1) -> Net-(C12-Pad2)
- U4 pad 2: Net-(C34-Pad1) -> Net-(C33-Pad1)
- U4 pad 3: Net-(C33-Pad1) -> Net-(C34-Pad1)
- U4 pad 5: Net-(C37-Pad1) -> Net-(C32-Pad1)
- U4 pad 6: Net-(C32-Pad1) -> Net-(C35-Pad2)
- U4 pad 7: Net-(C37-Pad1) -> Net-(C35-Pad2)
Routing:
- net +5V: track 247.3 -> 361.9 mm, vias 11 -> 19
- net -5V: track 216.5 -> 304.8 mm, vias 10 -> 15
- net /InputAmplifier/IN_AMP: track 14.0 -> 94.5 mm
- net GND: track 51.2 -> 98.8 mm, vias 75 -> 113
- net Net-(C35-Pad2): track 0.00 -> 30.3 mm, vias 0 -> 3
- net Net-(C79-Pad1): track 0.00 -> 26.4 mm, vias 0 -> 1
- net Net-(C68-Pad1): track 0.00 -> 26.4 mm, vias 0 -> 1
- net Net-(C57-Pad1): track 0.00 -> 26.4 mm, vias 0 -> 1
- net Net-(C24-Pad1): track 18.2 -> 41.2 mm, vias 0 -> 3
- net Net-(C12-Pad2): track 8.61 -> 26.4 mm, vias 0 -> 1
- net Net-(C12-Pad1): track 25.5 -> 9.52 mm, vias 0 -> 1
- net Net-(C37-Pad1): track 15.9 -> 0.00 mm
- net /GainBlock/GB_IN: track 31.7 -> 46.5 mm
- net /GainBlock/WB_OUT: track 17.0 -> 31.5 mm, vias 0 -> 2
- net Net-(C33-Pad1): track 29.3 -> 43.5 mm, vias 0 -> 3
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Other:
- board text added: "+5 GND GND -5"
- board text added: "1MHz"
- board text added: "4.99Ohm 49.9Ohm 499Ohm SHORT"
- board text added: "ABSOLUTE MAX 9V/2W"
- board text added: "JUMPERS"
- board text added: "POLARIZATION OF TANTALUM CAPS Removal of resistor ladder's pads"
- board text added: "PSU Noise tester 10Hz - 1MHz 80dB gain"
- board text added: "PWR ON"
- board text added: "WB"
- board text added: "github.com/PaulWozny/NoiseTester"
- board text removed: "1MHz OUT"
- board text removed: "POLARIZATION OF TANTALUM CAPS"
- board text removed: "WB OUT"

Commit message: BOM was updated
Parts:
- removed REF**: OSHW-Logo2_7.3x6mm_SilkScreen, Symbol:OSHW-Logo2_7.3x6mm_SilkScreen
- J2, J3, J5, J6: value Conn_Coaxial -> 5-1634503-1
- moved J6 0.14 mm to (99.4, 161.2), turned to 0 degrees
Connections:
- RN1 pad 2: /InputAmplifier/IN_AMP -> (no net)
- RN1 pad 7: /InputAmplifier/IN_AMP -> (no net)
- RN2 pad 2: /InputAmplifier/IN_AMP -> (no net)
- RN2 pad 7: /InputAmplifier/IN_AMP -> (no net)
- RN3 pad 2: /InputAmplifier/IN_AMP -> (no net)
- RN3 pad 7: /InputAmplifier/IN_AMP -> (no net)
- RN4 pad 2: /InputAmplifier/IN_AMP -> (no net)
- RN4 pad 7: /InputAmplifier/IN_AMP -> (no net)
Routing:
- net Net-(C43-Pad1): track 10.9 -> 12.8 mm
- net GND: vias 113 -> 120
Other:
- board text removed: "POLARIZATION OF TANTALUM CAPS Removal of resistor ladder's pads"
